Commit message: ros2 migration and update pr2 meshes

File: data/model.urdf (robot description, URDF)
Before this commit: robot 3d-coord-arrow-robot, 1 links, 0 joints
Links:
- link nil_link: geometry collision mesh filename=package://rviz_collada_marker/data/nil_link_mesh.dae scale=1 1 1; visual mesh filename=package://rviz_collada_marker/data/nil_link_mesh.dae scale=1 1 1

File: data/truck.urdf (robot description, URDF)
Before this commit: robot truck, 1 links, 0 joints
Links:
- removed link ego_frame
- added link /nil_link; visual mesh filename=package://rviz_collada_marker/data/truck.dae scale=1 1 1
